File: adapter/adapter.kicad_pcb (KiCad board)
At the start: 2 copper layers, 66 x 68.8 mm, 2 parts, among them J1 502078-1710, J2 Conn_01x18_Male

Commit message: re-routed
Routing:
- net /5: track 0.00 -> 55.0 mm, vias 0 -> 1
- net /13: track 0.00 -> 54.7 mm, vias 0 -> 1
- net /15: track 0.00 -> 52.8 mm, vias 0 -> 1
- net /9: track 0.00 -> 51.2 mm, vias 0 -> 1
- net /11: track 0.00 -> 49.0 mm, vias 0 -> 1
- net /7: track 0.00 -> 48.9 mm, vias 0 -> 1
- net /16: track 0.00 -> 46.3 mm
- net /14: track 0.00 -> 44.4 mm
- net /12: track 0.00 -> 42.5 mm
- net /10: track 0.00 -> 40.6 mm
- net /8: track 0.00 -> 40.5 mm, vias 1 -> 0
- net /6: track 6.08 -> 42.4 mm, vias 1 -> 0
- net /MP: track 60.6 -> 80.7 mm
- net /3: track 47.7 -> 52.8 mm, vias 0 -> 1
- net /2: track 46.2 -> 46.3 mm, vias 1 -> 0
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