File: main/main.kicad_pcb (KiCad board)
At the start: 2 copper layers, 70 parts, among them IC1 MAX14689EWL+T, IC2 MAX14689EWL+T, IC3 MAX14689EWL+T, IC4 MAX20303BEWN+, IC5 PAN1326B, J1 502078-1710, J2 DX07S024JJ3R1300, U1 MAX9062EBS+TG45, U2 MAX9062EBS+TG45, U3 MAX8532EBT2+T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

Commit message: renamed main. created board cuts
Parts:
- moved C25 47.7 mm to (194.8, 85.5)
- moved L2 47.7 mm to (211.0, 81.5)
- moved R1 47.7 mm to (208.0, 105.3)
- moved C1 47.7 mm to (210.9, 105.2)
- moved C10 47.7 mm to (224.9, 77.4)
- moved C11 47.7 mm to (220.8, 79.4)
- moved C12 47.7 mm to (222.0, 77.4)
- moved C13 47.7 mm to (214.7, 85.6)
- moved C14 47.7 mm to (211.8, 88.1)
- moved C15 47.7 mm to (214.7, 83.6)
- moved C16 47.7 mm to (217.9, 80.8)
- moved C18 47.7 mm to (214.7, 87.6)
- moved C19 47.7 mm to (217.6, 84.7)
- moved C2 47.7 mm to (218.1, 101.3)
- moved C20 47.7 mm to (217.6, 88.7)
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Other:
- board outline added: 18.3 x 35.6 mm

Commit message: update main board
Parts:
- J1: moved to B.Cu
- moved L2 116.9 mm to (94.2, 83.5)
- moved C10 116.9 mm to (108.1, 79.5)
- moved C11 116.9 mm to (103.9, 81.5)
- moved C12 116.9 mm to (105.2, 79.5)
- moved C13 116.9 mm to (97.9, 87.6)
- moved C14 116.9 mm to (95.0, 90.2)
- moved C15 116.9 mm to (97.9, 85.7)
- moved C16 116.9 mm to (101.1, 82.8)
- moved C17 116.9 mm to (103.9, 83.4)
- moved C18 116.9 mm to (97.9, 89.6)
- moved C19 116.9 mm to (100.8, 86.8)
- moved C20 116.9 mm to (100.8, 90.7)
- moved C21 116.9 mm to (106.8, 81.4)
- moved C5 116.9 mm to (100.8, 88.7)
- moved C6 116.9 mm to (97.9, 91.6)
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Other:
- board size 18.3 x 35.6 mm -> 18.3 x 36.1 mm

Commit message: added template data for printing
Parts:
- moved IC5 18.1 mm to (109.5, 104.6)
- moved S1 15.2 mm to (123.7, 109.7), turned to 90 degrees
- moved S2 6.61 mm to (143.0, 109.7), turned to 270 degrees
Other:
- copper layers 2 -> 6
