File: sensor/sensor.kicad_sch (KiCad schematic)
At the start: 44 parts, among them IC1 MAX30002CWV+, IC2 LP5900TLX-2.7_NOPB, IC3 MAX86141ENP+T, IC4 SIT1532AC, IC5 LP5900TLX-1.8_NOPB, J1 Conn_01x10_Female, J2 Conn_01x10_Female, J3 Probe_01_male, J4 Probe_01_male, J5 Probe_01_male, J6 Probe_01_male

Commit message: production update 2. added J1,J2 PN and changed via diameters
Parts:
- J1, J2: Manufacturer (none) -> Molex; Manufacturer Part Number (none) -> 90147-1110; Mouser part number (none) -> 538-90147-1110; Mouser parts/stock (none) -> https://www.mouser.ee/ProductDetail/Molex/90147-1110
- J3, J4, J5, J6: Manufacturer Part Number (none) -> 3977-1-00-15-00-00-03-0
